Commit message: gazebo compatibility

File: mycobot_description/urdf/mycobot.urdf (robot description, URDF)
Before this commit: robot firefighter, 8 links, 7 joints
Links:
- added link finger_left; visual mesh filename=package://mycobot_description/meshes/finger_left.stl scale=0.001 0.001 0.001
- added link finger_right; visual mesh filename=package://mycobot_description/meshes/finger_right.stl scale=0.001 0.001 0.001
- added link gripper_base; visual mesh filename=package://mycobot_description/meshes/gripper_base.stl scale=0.001 0.001 0.001
- added link tool0
- link joint6_flange: geometry visual cylinder length=0.014 radius=0.019
Joints:
- added joint ee_to_tool0: type fixed, parent joint6_flange, child tool0, origin xyz=0 0.062 0 rpy=0 0 1.5708
- added joint end_to_gripper_base: type fixed, parent joint6_flange, child gripper_base, origin xyz=0 0.007 0 rpy=0 0 1.5708, axis 0 0 1
- added joint gripper_base_to_l_finger: type prismatic, parent gripper_base, child finger_left, origin xyz=0.033 0 0 rpy=0 0 0, axis 0 1 0, limit lower=0 upper=0.018 effort=1.0 velocity=0
- added joint gripper_base_to_r_finger: type prismatic, parent gripper_base, child finger_right, origin xyz=0.033 0 0 rpy=0 0 0, axis 0 1 0, limit lower=-0.018 upper=0 effort=1.0 velocity=0, mimic joint=gripper_base_to_l_finger multiplier=-1
- joint base_mount_to_joint1: origin xyz=0 0 0 rpy=0 0 -1.5708 -> xyz=0 0 0.005 rpy=0 0 -1.5708
- joint joint6output_to_joint6: origin xyz=0 0.0456 0.03792  rpy=0 0 0 -> xyz=0 0.0526 0.03792  rpy=0 0 0
